Commit message: Kamera funktioniert jetzt richtig

File: install/ur10e_gazebo_sim/share/ur10e_gazebo_sim/urdf/camera_macro.xacro (robot description, xacro)
@@ -1,75 +1,77 @@
 <?xml version="1.0"?>
 <robot xmlns:xacro="http://ros.org/wiki/xacro">
-  <xacro:macro name="sensor_d435i_gazebo" params="parent prefix *origin">
-    <joint name="${prefix}camera_joint" type="fixed">
+  <xacro:macro name="sensor_d435i_gazebo" params="parent *origin">
+    <joint name="camera_joint" type="fixed">
       <xacro:insert_block name="origin" />
       <parent link="${parent}"/>
-      <child link="${prefix}camera_bottom_screw_frame" />
+      <child link="camera_bottom_screw_frame" />
     </joint>
-    <link name="${prefix}camera_bottom_screw_frame"/>
-    <joint name="${prefix}camera_link_joint" type="fixed">
+    <gazebo reference="camera_joint">
+        <disableFixedJointLumping>true</disableFixedJointLumping>
+        <preserveFixedJoint>true</preserveFixedJoint>
+    </gazebo>
+    <link name="camera_bottom_screw_frame">
+      <inertial>
+        <mass value="0.01" />
+        <origin xyz="0 0 0" />
+        <inertia ixx="0.0001" ixy="0" ixz="0" iyy="0.0001" iyz="0" izz="0.0001" />
+      </inertial>
+    </link>
+    <joint name="camera_link_joint" type="fixed">
       <origin xyz="0.0106 0.0175 0.0125" rpy="0 0 0"/>
-      <parent link="${prefix}camera_bottom_screw_frame"/>
-      <child link="${prefix}camera_link" />
+      <parent link="camera_bottom_screw_frame"/>
+      <child link="camera_link" />
     </joint>
-    <link name="${prefix}camera_link">
+    <gazebo reference="camera_link_joint">
+        <disableFixedJointLumping>true</disableFixedJointLumping>
+        <preserveFixedJoint>true</preserveFixedJoint>
+    </gazebo>
+    <link name="camera_link">
       <visual>
         <origin xyz="0 0 0" rpy="${pi/2} 0 ${pi/2}"/>
-        <geometry>
-          <mesh filename="package://realsense2_description/meshes/d435.dae" />
-        </geometry>
+        <geometry><mesh filename="package://realsense2_description/meshes/d435.dae" /></geometry>
       </visual>
       <collision>
         <origin xyz="0 -0.0175 0" rpy="0 0 0"/>
-        <geometry>
-          <box size="0.02505 0.090 0.025"/>
-        </geometry>
+        <geometry><box size="0.02505 0.090 0.025"/></geometry>
       </collision>
       <inertial>
         <mass value="0.072" />
         <origin xyz="0 0 0" />
-        <inertia ixx="0.003881243" ixy="0.0" ixz="0.0" iyy="0.000498940" iyz="0.0" izz="0.003879257" />
+        <inertia ixx="0.001" ixy="0" ixz="0" iyy="0.001" iyz="0" izz="0.001" />
       </inertial>
     </link>
-    <joint name="${prefix}camera_depth_joint" type="fixed">
+    <joint name="camera_depth_joint" type="fixed">
       <origin xyz="0 0 0" rpy="${-pi/2} 0 ${-pi/2}"/>
-      <parent link="${prefix}camera_link"/>
-      <child link="${prefix}camera_depth_frame" />
+      <parent link="camera_link"/>
+      <child link="camera_depth_frame" />
     </joint>
-    <link name="${prefix}camera_depth_frame"/>
-    <gazebo reference="${prefix}camera_link">
-      <sensor name="${prefix}d435i" type="depth">
+    <gazebo reference="camera_depth_joint">
+        <disableFixedJointLumping>true</disableFixedJointLumping>
+        <preserveFixedJoint>true</preserveFixedJoint>
+    </gazebo>
+    <link name="camera_depth_frame">
+      <inertial>
+        <mass value="0.001" /> <origin xyz="0 0 0" />
+        <inertia ixx="0.0001" ixy="0" ixz="0" iyy="0.0001" iyz="0" izz="0.0001" />
+      </inertial>
+    </link>
+    <gazebo reference="camera_link">
+      <sensor name="d435i" type="depth">
         <update_rate>30</update_rate>
+        <pose>0 0 0 0 0 0</pose>
         <camera>
-          <horizontal_fov>1.5184</horizontal_fov> <image>
-            <width>640</width>
-            <height>480</height>
-            <format>R8G8B8</format>
-          </image>
-          <clip>
-            <near>0.1</near>
-            <far>10.0</far>
-          </clip>
+          <horizontal_fov>1.5184</horizontal_fov>
+          <image><width>640</width><height>480</height><format>R8G8B8</format></image>
+          <clip><near>0.1</near><far>10.0</far></clip>
         </camera>
-        <plugin name="${prefix}camera_controller" filename="libgazebo_ros_camera.so">
-          <robotNamespace>/</robotNamespace>
-          <baseline>0.05</baseline>
-          <alwaysOn>true</alwaysOn>
-          <updateRate>30.0</updateRate>
-          <cameraName>${prefix}d435i</cameraName>
-          <imageTopicName>color/image_raw</imageTopicName>
-          <cameraInfoTopicName>color/camera_info</cameraInfoTopicName>
-          <depthImageTopicName>depth/image_rect_raw</depthImageTopicName>
-          <depthImageInfoTopicName>depth/camera_info</depthImageInfoTopicName>
-          <pointCloudTopicName>depth/color/points</pointCloudTopicName>
-          <frameName>${prefix}camera_depth_frame</frameName>
-          <pointCloudCutoff>0.1</pointCloudCutoff>
-          <pointCloudCutoffMax>10.0</pointCloudCutoffMax>
-          <hackBaseline>0.07</hackBaseline>
-          <distortionK1>0.0</distortionK1>
-          <distortionK2>0.0</distortionK2>
-          <distortionK3>0.0</distortionK3>
-          <distortionT1>0.0</distortionT1>
-          <distortionT2>0.0</distortionT2>
+        <plugin name="camera_controller" filename="libgazebo_ros_camera.so">
+          <ros>
+            </ros>
+          <camera_name>camera</camera_name>
+          <frame_name>camera_depth_frame</frame_name>
+          <hack_baseline>0.07</hack_baseline>
+          <min_depth>0.1</min_depth>
+          <max_depth>10.0</max_depth>
         </plugin>
       </sensor>

File: install/ur10e_gazebo_sim/share/ur10e_gazebo_sim/urdf/ur10e_ft_rg2.urdf.xacro (robot description, xacro)
@@ -57,5 +57,5 @@
      <link name="ground_plane">
        <visual>
-         <origin rpy="0 0 0" xyz="0 0 0"/>
+         <origin rpy="0 0 0" xyz="0 0 0.927"/>
          <geometry>
            <box size="5 5 0"/>
@@ -66,5 +66,5 @@
        </visual>
        <collision>
-         <origin rpy="0 0 0" xyz="0 0 0"/>
+         <origin rpy="0 0 0" xyz="0 0 0.927"/>
          <geometry>
            <box size="5 5 0"/>
@@ -118,6 +118,24 @@
      <origin xyz="1.31950 0.57082 0.927" rpy="0 0 0" />          <!-- position robot in the world -->
    </xacro:ur_robot>
-    <xacro:sensor_d435i_gazebo parent="tool0" prefix="camera_">
-      <origin xyz="0.019 -0.07 0" rpy="1.57 -1.57 0"/>    <!-- Kamera Position und Orientierung-->
+    <link name="camera_mount_link">
+      <!-- <visual>
+        <geometry><box size="0.05 0.05 0.05"/></geometry>
+        <material name="red"><color rgba="1 0 0 1"/></material>
+      </visual>
+      <collision>
+        <geometry><box size="0.05 0.05 0.05"/></geometry>
+      </collision> -->
+      <inertial>
+        <mass value="0.1" /> <origin xyz="0 0 0" />
+        <inertia ixx="0.001" ixy="0" ixz="0" iyy="0.001" iyz="0" izz="0.001" />
+      </inertial>
+    </link>
+    <joint name="wrist_to_mount_joint" type="fixed">
+      <parent link="wrist_3_link" />
+      <child link="camera_mount_link" />
+      <origin xyz="0.019 -0.07 0.015" rpy="1.57 -1.57 0" />
+    </joint>
+    <xacro:sensor_d435i_gazebo parent="camera_mount_link">
+      <origin xyz="0 0 0" rpy="0 0 0"/>
     </xacro:sensor_d435i_gazebo>
    <xacro:if value="$(arg sim_gazebo)">
