Commit message: Setup in Gazebo eingebaut

File: install/ur10e_gazebo_sim/share/ur10e_gazebo_sim/urdf/ur10e_ft_rg2.urdf.xacro (robot description, xacro)
@@ -116,5 +116,5 @@
      trajectory_port="$(arg trajectory_port)"
      >
-     <origin xyz="1.31950 0.57082 0.927" rpy="0 0 0" />          <!-- position robot in the world -->
+     <origin xyz="1.65 0.865 0.927" rpy="0 0 0" />          <!-- position robot in the world: x = red y = green x = blue(height) -->
    </xacro:ur_robot>
     <link name="camera_mount_link">
