Commit message: Roboter spawned in Gazebo auf dem Setup

File: install/ur10e_ft_rg2_moveit_config/share/ur10e_ft_rg2_moveit_config/config/ur.ros2_control.xacro (robot description, xacro)
@@ -1,61 +1 @@
-<?xml version="1.0"?>
-<robot xmlns:xacro="http://www.ros.org/wiki/xacro">
-    <xacro:macro name="ur_ros2_control" params="name initial_positions_file">
-        <xacro:property name="initial_positions" value="${load_yaml(initial_positions_file)['initial_positions']}"/>
-        <ros2_control name="${name}" type="system">
-            <hardware>
-                <!-- By default, set up controllers for simulation. This won't work on real hardware -->
-                <plugin>mock_components/GenericSystem</plugin>
-            </hardware>
-            <joint name="shoulder_pan_joint">
-                <command_interface name="position"/>
-                <state_interface name="position">
-                  <param name="initial_value">${initial_positions['shoulder_pan_joint']}</param>
-                </state_interface>
-                <state_interface name="velocity"/>
-            </joint>
-            <joint name="shoulder_lift_joint">
-                <command_interface name="position"/>
-                <state_interface name="position">
-                  <param name="initial_value">${initial_positions['shoulder_lift_joint']}</param>
-                </state_interface>
-                <state_interface name="velocity"/>
-            </joint>
-            <joint name="elbow_joint">
-                <command_interface name="position"/>
-                <state_interface name="position">
-                  <param name="initial_value">${initial_positions['elbow_joint']}</param>
-                </state_interface>
-                <state_interface name="velocity"/>
-            </joint>
-            <joint name="wrist_1_joint">
-                <command_interface name="position"/>
-                <state_interface name="position">
-                  <param name="initial_value">${initial_positions['wrist_1_joint']}</param>
-                </state_interface>
-                <state_interface name="velocity"/>
-            </joint>
-            <joint name="wrist_2_joint">
-                <command_interface name="position"/>
-                <state_interface name="position">
-                  <param name="initial_value">${initial_positions['wrist_2_joint']}</param>
-                </state_interface>
-                <state_interface name="velocity"/>
-            </joint>
-            <joint name="wrist_3_joint">
-                <command_interface name="position"/>
-                <state_interface name="position">
-                  <param name="initial_value">${initial_positions['wrist_3_joint']}</param>
-                </state_interface>
-                <state_interface name="velocity"/>
-            </joint>
-            <joint name="rg2_gripper_finger_joint">
-                <command_interface name="position"/>
-                <state_interface name="position">
-                  <param name="initial_value">${initial_positions['rg2_gripper_finger_joint']}</param>
-                </state_interface>
-                <state_interface name="velocity"/>
-            </joint>
-        </ros2_control>
-    </xacro:macro>
-</robot>
+/home/matteo-melzer/gazebo_test/src/ur10e_ft_rg2_moveit_config/config/ur.ros2_control.xacro

File: install/ur10e_ft_rg2_moveit_config/share/ur10e_ft_rg2_moveit_config/config/ur.urdf.xacro (robot description, xacro)
@@ -1,9 +1 @@
-<?xml version="1.0"?>
-<robot xmlns:xacro="http://www.ros.org/wiki/xacro" name="ur">
-    <!-- <xacro:arg name="initial_positions_file" default="initial_positions.yaml" /> -->
-    <!-- Import ur urdf file -->
-    <xacro:include filename="$(find ur10e_gazebo_sim)/urdf/ur10e_ft_rg2.urdf.xacro" />
-    <!-- Import control_xacro -->
-    <!-- <xacro:include filename="ur.ros2_control.xacro" /> -->
-    <!-- <xacro:ur_ros2_control name="FakeSystem" initial_positions_file="$(arg initial_positions_file)"/> -->
-</robot>
+/home/matteo-melzer/gazebo_test/src/ur10e_ft_rg2_moveit_config/config/ur.urdf.xacro

File: install/ur10e_gazebo_sim/share/ur10e_gazebo_sim/urdf/ur10e_flex.urdf.xacro (robot description, xacro)
@@ -5,4 +5,5 @@
    <!-- import main macro -->
    <xacro:include filename="$(find ur10e_gazebo_sim)/urdf/ur10e_macro.xacro"/>
+   <xacro:include filename="$(find ur10e_gazebo_sim)/urdf/camera_macro.xacro"/>
    <!-- possible 'ur_type' values: ur3, ur5, ur10, ur3e, ur5e, ur7e, ur10e, ur12e, ur16e, ur8long, ur15, ur18, ur20, ur30 -->
    <!-- the default value should raise an error in case this was called without defining the type -->
@@ -115,6 +116,9 @@
      trajectory_port="$(arg trajectory_port)"
      >
-     <origin xyz="0 0 0.01" rpy="0 0 0" />          <!-- position robot in the world -->
+     <origin xyz="1.31950 0.57082 0.927" rpy="0 0 0" />          <!-- position robot in the world -->
    </xacro:ur_robot>
+   <xacro:sensor_d435i_gazebo parent="tool0" prefix="camera_">
+      <origin xyz="0.019 -0.07 0" rpy="1.57 -1.57 0"/>    <!-- Kamera Position und Orientierung-->
+    </xacro:sensor_d435i_gazebo>
    <xacro:if value="$(arg sim_gazebo)">
     <!-- Gazebo plugins -->

File: install/ur10e_gazebo_sim/share/ur10e_gazebo_sim/urdf/ur10e_ft_rg2.urdf.xacro (robot description, xacro)
@@ -5,4 +5,5 @@
    <!-- import main macro -->
    <xacro:include filename="$(find ur10e_gazebo_sim)/urdf/ur10e_macro.xacro"/>
+   <xacro:include filename="$(find ur10e_gazebo_sim)/urdf/camera_macro.xacro"/>
    <!-- possible 'ur_type' values: ur3, ur5, ur10, ur3e, ur5e, ur7e, ur10e, ur12e, ur16e, ur8long, ur15, ur18, ur20, ur30 -->
    <!-- the default value should raise an error in case this was called without defining the type -->
@@ -115,6 +116,9 @@
      trajectory_port="$(arg trajectory_port)"
      >
-     <origin xyz="0 0 0.01" rpy="0 0 0" />          <!-- position robot in the world -->
+     <origin xyz="1.31950 0.57082 0.927" rpy="0 0 0" />          <!-- position robot in the world -->
    </xacro:ur_robot>
+    <xacro:sensor_d435i_gazebo parent="tool0" prefix="camera_">
+      <origin xyz="0.019 -0.07 0" rpy="1.57 -1.57 0"/>    <!-- Kamera Position und Orientierung-->
+    </xacro:sensor_d435i_gazebo>
    <xacro:if value="$(arg sim_gazebo)">
     <!-- Gazebo plugins -->
